File: pcb files/lightnincontroller pcb/RTC.sch (KiCad schematic (older format))
At the start: 11 parts

Commit message: lightning controller
lightining controller allen neopixels af te tekenen +voeding
Parts:
- BT1: renamed from BT?; footprint (none) -> Battery:BatteryHolder_Keystone_3008_1x2450
- C13, C14, C15, C16: renamed from C?; footprint (none) -> Capacitor_SMD:C_0603_1608Metric
- R7, R8: renamed from R?; footprint (none) -> Resistor_SMD:R_0603_1608Metric
- TP7, TP8: renamed from TP?; footprint (none) -> Connector_PinSocket_2.54mm:PinSocket_1x01_P2.54mm_Vertical
- Y3: renamed from Y?; footprint (none) -> Crystal:Crystal_DS15_D1.5mm_L5.0mm_Horizontal
- gave numbers to parts that had none: 1
Changed lines of the file:
@@
 $Descr A4 11693 8268
 encoding utf-8
-Sheet 4 4
+Sheet 4 5
 Title ""
 Date ""
@@
 $EndDescr
 $Comp
-L Timer_RTC:DS1307N+ U?
+L Timer_RTC:DS1307N+ U3
 U 1 1 5BD55C10
 P 3270 4630
-F 0 "U?" H 3120 4630 50  0000 L CNN
+F 0 "U3" H 3120 4630 50  0000 L CNN
 F 1 "DS1307N+" H 3380 4970 50  0000 L CNN
 F 2 "Package_DIP:DIP-8_W7.62mm" H 3270 4130 50  0001 C CNN
@@
 $EndComp
 $Comp
-L Device:Battery_Cell BT?
+L Device:Battery_Cell BT1
 U 1 1 5BD49479
-P 1330 4750
-F 0 "BT?" H 1448 4846 50  0000 L CNN
-F 1 "Battery_Cell" H 1448 4755 50  0000 L CNN
-F 2 "" V 1330 4810 50  0001 C CNN
-F 3 "~" V 1330 4810 50  0001 C CNN
-	1    1330 4750
-	1    0    0    -1
-$EndComp
-$Comp
-L power:+BATT #PWR?
+P 1290 4410
+F 0 "BT1" H 1408 4506 50  0000 L CNN
+F 1 "Battery_Cell" H 1408 4415 50  0000 L CNN
+F 2 "Battery:BatteryHolder_Keystone_3008_1x2450" V 1290 4470 50  0001 C CNN
+F 3 "~" V 1290 4470 50  0001 C CNN
+	1    1290 4410
+	1    0    0    -1
+$EndComp
+$Comp
+L power:+BATT #PWR0131
 U 1 1 5BD4950E
-P 1330 4550
-F 0 "#PWR?" H 1330 4400 50  0001 C CNN
-F 1 "+BATT" H 1345 4723 50  0000 C CNN
-F 2 "" H 1330 4550 50  0001 C CNN
-F 3 "" H 1330 4550 50  0001 C CNN
-	1    1330 4550
-	1    0    0    -1
-$EndComp
-$Comp
-L power:+BATT #PWR?
+P 1290 4210
+F 0 "#PWR0131" H 1290 4060 50  0001 C CNN
+F 1 "+BATT" H 1305 4383 50  0000 C CNN
+F 2 "" H 1290 4210 50  0001 C CNN
+F 3 "" H 1290 4210 50  0001 C CNN
+	1    1290 4210
+	1    0    0    -1
+$EndComp
+$Comp
+L power:+BATT #PWR0132
 U 1 1 5BD4952E
 P 3270 3870
-F 0 "#PWR?" H 3270 3720 50  0001 C CNN
+F 0 "#PWR0132" H 3270 3720 50  0001 C CNN
 F 1 "+BATT" H 3285 4043 50  0000 C CNN
 F 2 "" H 3270 3870 50  0001 C CNN
@@
 $EndComp
 $Comp
-L power:+3V3 #PWR?
+L power:+3V3 #PWR0133
 U 1 1 5BD49570
 P 3370 4050
-F 0 "#PWR?" H 3370 3900 50  0001 C CNN
+F 0 "#PWR0133" H 3370 3900 50  0001 C CNN
 F 1 "+3V3" H 3385 4223 50  0000 C CNN
 F 2 "" H 3370 4050 50  0001 C CNN
@@
 	3370 4230 3370 4050
 $Comp
-L power:GND #PWR?
+L power:GND #PWR0134
 U 1 1 5BD49607
-P 1330 4850
-F 0 "#PWR?" H 1330 4600 50  0001 C CNN
-F 1 "GND" H 1335 4677 50  0000 C CNN
-F 2 "" H 1330 4850 50  0001 C CNN
-F 3 "" H 1330 4850 50  0001 C CNN
-	1    1330 4850
-	1    0    0    -1
-$EndComp
-$Comp
-L power:GND #PWR?
+P 1290 4510
+F 0 "#PWR0134" H 1290 4260 50  0001 C CNN
+F 1 "GND" H 1295 4337 50  0000 C CNN
+F 2 "" H 1290 4510 50  0001 C CNN
+F 3 "" H 1290 4510 50  0001 C CNN
+	1    1290 4510
+	1    0    0    -1
+$EndComp
+$Comp
+L power:GND #PWR0135
 U 1 1 5BD49625
 P 3270 5030
-F 0 "#PWR?" H 3270 4780 50  0001 C CNN
+F 0 "#PWR0135" H 3270 4780 50  0001 C CNN
 F 1 "GND" H 3275 4857 50  0000 C CNN
 F 2 "" H 3270 5030 50  0001 C CNN
@@
 $EndComp
 $Comp
-L Device:Crystal Y?
+L Device:Crystal Y3
 U 1 1 5BD4A339
 P 4330 4940
-F 0 "Y?" V 4376 4809 50  0000 R CNN
+F 0 "Y3" V 4376 4809 50  0000 R CNN
 F 1 "Crystal" V 4285 4809 50  0000 R CNN
-F 2 "" H 4330 4940 50  0001 C CNN
+F 2 "Crystal:Crystal_DS15_D1.5mm_L5.0mm_Horizontal" H 4330 4940 50  0001 C CNN
 F 3 "~" H 4330 4940 50  0001 C CNN
 	1    4330 4940
@@
 	3770 4530 4860 4530
 $Comp
-L Device:R R?
+L Device:R R7
 U 1 1 5BD4A5C9
 P 3960 4280
-F 0 "R?" H 4030 4326 50  0000 L CNN
+F 0 "R7" H 4030 4326 50  0000 L CNN
 F 1 "R" H 4030 4235 50  0000 L CNN
-F 2 "" V 3890 4280 50  0001 C CNN
+F 2 "Resistor_SMD:R_0603_1608Metric" V 3890 4280 50  0001 C CNN
 F 3 "~" H 3960 4280 50  0001 C CNN
 	1    3960 4280
@@
 	3960 4430 4190 4430
 $Comp
-L Device:R R?
+L Device:R R8
 U 1 1 5BD4A629
 P 4860 4380
-F 0 "R?" H 4930 4426 50  0000 L CNN
+F 0 "R8" H 4930 4426 50  0000 L CNN
 F 1 "R" H 4930 4335 50  0000 L CNN
-F 2 "" V 4790 4380 50  0001 C CNN
+F 2 "Resistor_SMD:R_0603_1608Metric" V 4790 4380 50  0001 C CNN
 F 3 "~" H 4860 4380 50  0001 C CNN
 	1    4860 4380
@@
 Connection ~ 4860 4530
 $Comp
-L power:+3V3 #PWR?
+L power:+3V3 #PWR0136
 U 1 1 5BD4A6DA
 P 3960 4130
-F 0 "#PWR?" H 3960 3980 50  0001 C CNN
+F 0 "#PWR0136" H 3960 3980 50  0001 C CNN
 F 1 "+3V3" H 3975 4303 50  0000 C CNN
 F 2 "" H 3960 4130 50  0001 C CNN
@@
 $EndComp
 $Comp
-L power:+3V3 #PWR?
+L power:+3V3 #PWR0137
 U 1 1 5BD4A6EF
 P 4860 4230
-F 0 "#PWR?" H 4860 4080 50  0001 C CNN
+F 0 "#PWR0137" H 4860 4080 50  0001 C CNN
 F 1 "+3V3" H 4875 4403 50  0000 C CNN
 F 2 "" H 4860 4230 50  0001 C CNN
@@
 SDA
 $Comp
-L Connector:Test_Point TP?
+L Connector:Test_Point TP7
 U 1 1 5BD4A772
 P 4190 4430
-F 0 "TP?" H 4248 4550 50  0000 L CNN
+F 0 "TP7" H 4248 4550 50  0000 L CNN
 F 1 "Test_Point" H 4190 4630 50  0000 L CNN
-F 2 "" H 4390 4430 50  0001 C CNN
+F 2 "Connector_PinSocket_2.54mm:PinSocket_1x01_P2.54mm_Vertical" H 4390 4430 50  0001 C CNN
 F 3 "~" H 4390 4430 50  0001 C CNN
 	1    4190 4430
@@
 	4190 4430 4530 4430
 $Comp
-L Connector:Test_Point TP?
+L Connector:Test_Point TP8
 U 1 1 5BD4A7D0
 P 5270 4530
-F 0 "TP?" H 5328 4650 50  0000 L CNN
+F 0 "TP8" H 5328 4650 50  0000 L CNN
 F 1 "Test_Point" H 5270 4730 50  0000 L CNN
-F 2 "" H 5470 4530 50  0001 C CNN
+F 2 "Connector_PinSocket_2.54mm:PinSocket_1x01_P2.54mm_Vertical" H 5470 4530 50  0001 C CNN
 F 3 "~" H 5470 4530 50  0001 C CNN
 	1    5270 4530
@@
 NoConn ~ 2770 4630
 $Comp
-L power:+BATT #PWR?
+L power:+BATT #PWR0138
 U 1 1 5BD4AAA8
 P 1610 5590
-F 0 "#PWR?" H 1610 5440 50  0001 C CNN
+F 0 "#PWR0138" H 1610 5440 50  0001 C CNN
 F 1 "+BATT" H 1625 5763 50  0000 C CNN
 F 2 "" H 1610 5590 50  0001 C CNN
@@
 $EndComp
 $Comp
-L power:GND #PWR?
+L power:GND #PWR0139
 U 1 1 5BD4AAC1
 P 1590 6010
-F 0 "#PWR?" H 1590 5760 50  0001 C CNN
+F 0 "#PWR0139" H 1590 5760 50  0001 C CNN
 F 1 "GND" H 1595 5837 50  0000 C CNN
 F 2 "" H 1590 6010 50  0001 C CNN
@@
 $EndComp
 $Comp
-L Device:C_Small C?
+L Device:C_Small C13
 U 1 1 5BD4AB1B
 P 1490 5840
-F 0 "C?" H 1398 5794 50  0000 R CNN
+F 0 "C13" H 1398 5794 50  0000 R CNN
 F 1 "C_Small" H 1398 5885 50  0000 R CNN
-F 2 "" H 1490 5840 50  0001 C CNN
+F 2 "Capacitor_SMD:C_0603_1608Metric" H 1490 5840 50  0001 C CNN
 F 3 "~" H 1490 5840 50  0001 C CNN
 	1    1490 5840
@@
 $EndComp
 $Comp
-L Device:C_Small C?
+L Device:C_Small C14
 U 1 1 5BD4AB8E
 P 1700 5840
-F 0 "C?" H 1792 5886 50  0000 L CNN
+F 0 "C14" H 1792 5886 50  0000 L CNN
 F 1 "C_Small" H 1792 5795 50  0000 L CNN
-F 2 "" H 1700 5840 50  0001 C CNN
+F 2 "Capacitor_SMD:C_0603_1608Metric" H 1700 5840 50  0001 C CNN
 F 3 "~" H 1700 5840 50  0001 C CNN
 	1    1700 5840
@@
 $EndComp
 $Comp
-L power:+3V3 #PWR?
+L power:+3V3 #PWR0140
 U 1 1 5BD4ABD2
 P 2660 5590
-F 0 "#PWR?" H 2660 5440 50  0001 C CNN
+F 0 "#PWR0140" H 2660 5440 50  0001 C CNN
 F 1 "+3V3" H 2675 5763 50  0000 C CNN
 F 2 "" H 2660 5590 50  0001 C CNN
@@
 $EndComp
 $Comp
-L Device:C_Small C?
+L Device:C_Small C15
 U 1 1 5BD4ABEF
 P 2520 5850
-F 0 "C?" H 2428 5804 50  0000 R CNN
+F 0 "C15" H 2428 5804 50  0000 R CNN
 F 1 "C_Small" H 2428 5895 50  0000 R CNN
-F 2 "" H 2520 5850 50  0001 C CNN
+F 2 "Capacitor_SMD:C_0603_1608Metric" H 2520 5850 50  0001 C CNN
 F 3 "~" H 2520 5850 50  0001 C CNN
 	1    2520 5850
@@
 $EndComp
 $Comp
-L Device:C_Small C?
+L Device:C_Small C16
 U 1 1 5BD4AC45
 P 2830 5850
-F 0 "C?" H 2922 5896 50  0000 L CNN
+F 0 "C16" H 2922 5896 50  0000 L CNN
 F 1 "C_Small" H 2922 5805 50  0000 L CNN
-F 2 "" H 2830 5850 50  0001 C CNN
+F 2 "Capacitor_SMD:C_0603_1608Metric" H 2830 5850 50  0001 C CNN
 F 3 "~" H 2830 5850 50  0001 C CNN
 	1    2830 5850
@@
 	2660 5590 2830 5590
 $Comp
-L power:GND #PWR?
+L power:GND #PWR0141
 U 1 1 5BD4B14C
 P 2670 5960
-F 0 "#PWR?" H 2670 5710 50  0001 C CNN
+F 0 "#PWR0141" H 2670 5710 50  0001 C CNN
 F 1 "GND" H 2675 5787 50  0000 C CNN
 F 2 "" H 2670 5960 50  0001 C CNN

Commit message: 7833
voeding en  neopixls verbeterd
Parts:
- added TP9: Test_Point, Connector_PinSocket_2.54mm:PinSocket_1x01_P2.54mm_Vertical, symbol Connector:Test_Point
Connections:
- wire segments 28 -> 30
- no-connect marks 1 -> 0
Changed lines of the file:
@@
 Wire Wire Line
 	5270 4530 5580 4530
-NoConn ~ 2770 4630
 $Comp
 L power:+BATT #PWR0138
@@
 	1700 5590 1610 5590
 Connection ~ 1610 5590
+$Comp
+L Connector:Test_Point TP9
+U 1 1 5BFE88D7
+P 2440 4570
+F 0 "TP9" H 2498 4690 50  0000 L CNN
+F 1 "Test_Point" H 2440 4770 50  0000 L CNN
+F 2 "Connector_PinSocket_2.54mm:PinSocket_1x01_P2.54mm_Vertical" H 2640 4570 50  0001 C CNN
+F 3 "~" H 2640 4570 50  0001 C CNN
+	1    2440 4570
+	1    0    0    -1
+$EndComp
+Wire Wire Line
+	2770 4630 2440 4630
+Wire Wire Line
+	2440 4630 2440 4570
 $EndSCHEMATC
