File: pcb files/lightnincontroller pcb/ESP8266.sch (KiCad schematic (older format))
At the start: 18 parts

Commit message: lightning controller
lightining controller allen neopixels af te tekenen +voeding
Parts:
- C10, C11, C12, C7, C8, C9: renamed from C?; footprint (none) -> Capacitor_SMD:C_0603_1608Metric
- R4, R5, R6: renamed from R?; footprint (none) -> Resistor_SMD:R_0603_1608Metric
- TP1, TP2, TP3, TP4, TP5, TP6: renamed from TP?; footprint (none) -> Connector_PinSocket_2.54mm:PinSocket_1x01_P2.54mm_Vertical
- U2: renamed from U?; footprint (none) -> Package_SO:SSOP-16_4.4x5.2mm_P0.65mm
- Y2: renamed from Y?; footprint (none) -> Crystal:Crystal_HC33-U_Vertical
- gave numbers to parts that had none: 1

Commit message: 3de bodys toegevoed
pcb 3d view body;s toegevoegd
Parts:
- added TP10, TP7, TP8, TP9: Test_Point, Connector_PinSocket_2.54mm:PinSocket_1x01_P2.54mm_Vertical, symbol Connector:Test_Point
- Y2: footprint Crystal:Crystal_HC33-U_Vertical -> Crystal:Crystal_HC49-U_Horizontal
Connections:
- wire segments 55 -> 62
Changed lines of the file:
@@
 	1650 3690 1960 3690
 Wire Wire Line
-	1650 3490 2040 3490
-Wire Wire Line
-	1650 3390 2050 3390
-Wire Wire Line
-	1650 3290 2050 3290
-Wire Wire Line
-	1650 3190 2050 3190
-Wire Wire Line
 	1650 2990 2040 2990
-Text HLabel 2050 3190 2    50   Input ~ 0
+Text HLabel 2640 3190 2    50   Input ~ 0
 GPIO_0
-Text HLabel 2050 3290 2    50   Input ~ 0
+Text HLabel 2650 3290 2    50   Input ~ 0
 RTS
-Text HLabel 2050 3390 2    50   Input ~ 0
+Text HLabel 2650 3390 2    50   Input ~ 0
 GPIO2
-Text HLabel 2040 3490 2    50   Input ~ 0
+Text HLabel 2650 3490 2    50   Input ~ 0
 CH_PD
 Text Label 2040 2990 2    50   ~ 0
@@
 F 0 "Y2" H 2860 1528 50  0000 C CNN
 F 1 "Crystal" H 2860 1437 50  0000 C CNN
-F 2 "Crystal:Crystal_HC33-U_Vertical" H 2860 1260 50  0001 C CNN
+F 2 "Crystal:Crystal_HC49-U_Horizontal" H 2860 1260 50  0001 C CNN
 F 3 "~" H 2860 1260 50  0001 C CNN
 	1    2860 1260
@@
 	1280 4640 1170 4640
 Connection ~ 1170 4640
+Wire Wire Line
+	1650 3190 2270 3190
+Wire Wire Line
+	1650 3290 2380 3290
+Wire Wire Line
+	1650 3390 2460 3390
+Wire Wire Line
+	1650 3490 2570 3490
+$Comp
+L Connector:Test_Point TP7
+U 1 1 5C203D35
+P 2270 3190
+F 0 "TP7" V 2270 3370 50  0000 L CNN
+F 1 "Test_Point" H 2328 3219 50  0001 L CNN
+F 2 "Connector_PinSocket_2.54mm:PinSocket_1x01_P2.54mm_Vertical" H 2470 3190 50  0001 C CNN
+F 3 "~" H 2470 3190 50  0001 C CNN
+	1    2270 3190
+	1    0    0    -1
+$EndComp
+Connection ~ 2270 3190
+Wire Wire Line
+	2270 3190 2640 3190
+$Comp
+L Connector:Test_Point TP8
+U 1 1 5C203E2E
+P 2380 3030
+F 0 "TP8" V 2380 3210 50  0000 L CNN
+F 1 "Test_Point" H 2438 3059 50  0001 L CNN
+F 2 "Connector_PinSocket_2.54mm:PinSocket_1x01_P2.54mm_Vertical" H 2580 3030 50  0001 C CNN
+F 3 "~" H 2580 3030 50  0001 C CNN
+	1    2380 3030
+	1    0    0    -1
+$EndComp
+$Comp
+L Connector:Test_Point TP9
+U 1 1 5C203F6C
+P 2460 2870
+F 0 "TP9" V 2460 3050 50  0000 L CNN
+F 1 "Test_Point" H 2518 2899 50  0001 L CNN
+F 2 "Connector_PinSocket_2.54mm:PinSocket_1x01_P2.54mm_Vertical" H 2660 2870 50  0001 C CNN
+F 3 "~" H 2660 2870 50  0001 C CNN
+	1    2460 2870
+	1    0    0    -1
+$EndComp
+$Comp
+L Connector:Test_Point TP10
+U 1 1 5C20407F
+P 2570 2780
+F 0 "TP10" V 2570 2960 50  0000 L CNN
+F 1 "Test_Point" H 2628 2809 50  0001 L CNN
+F 2 "Connector_PinSocket_2.54mm:PinSocket_1x01_P2.54mm_Vertical" H 2770 2780 50  0001 C CNN
+F 3 "~" H 2770 2780 50  0001 C CNN
+	1    2570 2780
+	1    0    0    -1
+$EndComp
+Wire Wire Line
+	2380 3030 2380 3290
+Connection ~ 2380 3290
+Wire Wire Line
+	2380 3290 2650 3290
+Wire Wire Line
+	2460 3390 2460 2870
+Connection ~ 2460 3390
+Wire Wire Line
+	2460 3390 2650 3390
+Wire Wire Line
+	2570 2780 2570 3490
+Connection ~ 2570 3490
+Wire Wire Line
+	2570 3490 2650 3490
 $EndSCHEMATC

Commit message: pic
pic controller en co gerouted
Parts:
- Y2: footprint Crystal:Crystal_HC49-U_Horizontal -> Crystal:Crystal_HC49-4H_Vertical
Changed lines of the file:
@@
 F 0 "Y2" H 2860 1528 50  0000 C CNN
 F 1 "Crystal" H 2860 1437 50  0000 C CNN
-F 2 "Crystal:Crystal_HC49-U_Horizontal" H 2860 1260 50  0001 C CNN
+F 2 "Crystal:Crystal_HC49-4H_Vertical" H 2860 1260 50  0001 C CNN
 F 3 "~" H 2860 1260 50  0001 C CNN
 	1    2860 1260
