File: pcb files/lightnincontroller pcb/controller.sch (KiCad schematic (older format))
At the start: 10 parts

Commit message: schemerdetectie
schemerdetectie toegevoegd
Connections:
- net labels added: CH_PD, GPIO0, GPIO2, PhotoCel, RST
- no-connect marks 0 -> 6
Other:
- note added: "TX en RX op aparte I2C to uart chip\n"
Changed lines of the file:
@@
 Comment4 ""
 $EndDescr
-$Comp
-L Halfgelijders:PIC32MX170F256B-I_SP U?
-U 1 1 5BC35CAF
-P 3960 3560
-F 0 "U?" H 6110 6425 50  0000 C CNN
-F 1 "PIC32MX170F256B-I_SP" H 6110 6334 50  0000 C CNN
-F 2 "SeeedOPL-IC-2016:DIP28-2.54-34.7X7.62MM" H 3960 3560 50  0001 C CNN
-F 3 "" H 3960 3560 50  0001 C CNN
-	1    3960 3560
-	1    0    0    -1
-$EndComp
 Text HLabel 3220 1860 0    50   Input ~ 0
 SCL
@@
 Wire Wire Line
 	2970 5620 3070 5620
+Text HLabel 8460 1310 2    50   Input ~ 0
+PhotoCel
+NoConn ~ 3760 1110
+NoConn ~ 3760 1260
+NoConn ~ 3760 2460
+NoConn ~ 3760 2610
+NoConn ~ 3760 2910
+$Comp
+L Halfgelijders:PIC32MX170F256B-I_SP U?
+U 1 1 5BC35CAF
+P 3960 3560
+F 0 "U?" H 6110 6425 50  0000 C CNN
+F 1 "PIC32MX170F256B-I_SP" H 6110 6334 50  0000 C CNN
+F 2 "SeeedOPL-IC-2016:DIP28-2.54-34.7X7.62MM" H 3960 3560 50  0001 C CNN
+F 3 "" H 3960 3560 50  0001 C CNN
+	1    3960 3560
+	1    0    0    -1
+$EndComp
+NoConn ~ 4780 -15560
+Text Notes 4040 660  0    50   ~ 0
+TX en RX op aparte I2C to uart chip\n
+Text HLabel 8460 1460 2    50   Input ~ 0
+CH_PD
+Text HLabel 8460 1610 2    50   Input ~ 0
+GPIO2
+Text HLabel 8460 1760 2    50   Input ~ 0
+RST
+Text HLabel 8460 1910 2    50   Input ~ 0
+GPIO0
+Text Notes 2990 -470 0    50   ~ 0
+TX en RX op aparte I2C to uart chip\n
 $EndSCHEMATC

Commit message: esp en ds1307
gestart aan ds1307 interface
Connections:
- net labels added: RESET, ~IRQ
- wire segments 32 -> 34
- no-connect marks 6 -> 4
Changed lines of the file:
@@
 $Descr A4 11693 8268
 encoding utf-8
-Sheet 2 2
+Sheet 2 4
 Title ""
-Date ""
-Rev ""
+Date "2018-10-27"
+Rev "V0"
 Comp ""
 Comment1 ""
@@
 NoConn ~ 3760 1110
 NoConn ~ 3760 1260
-NoConn ~ 3760 2460
-NoConn ~ 3760 2610
 NoConn ~ 3760 2910
-$Comp
-L Halfgelijders:PIC32MX170F256B-I_SP U?
-U 1 1 5BC35CAF
-P 3960 3560
-F 0 "U?" H 6110 6425 50  0000 C CNN
-F 1 "PIC32MX170F256B-I_SP" H 6110 6334 50  0000 C CNN
-F 2 "SeeedOPL-IC-2016:DIP28-2.54-34.7X7.62MM" H 3960 3560 50  0001 C CNN
-F 3 "" H 3960 3560 50  0001 C CNN
-	1    3960 3560
-	1    0    0    -1
-$EndComp
 NoConn ~ 4780 -15560
 Text Notes 4040 660  0    50   ~ 0
@@
 Text Notes 2990 -470 0    50   ~ 0
 TX en RX op aparte I2C to uart chip\n
+Wire Wire Line
+	3760 2460 3570 2460
+Text HLabel 3570 2460 0    50   Input ~ 0
+~IRQ
+Wire Wire Line
+	3760 2610 3550 2610
+Text HLabel 3550 2610 0    50   Input ~ 0
+RESET
+$Comp
+L Halfgelijders:PIC32MX170F256B-I_SP U?
+U 1 1 5BC35CAF
+P 3960 3560
+F 0 "U?" H 6110 6425 50  0000 C CNN
+F 1 "PIC32MX170F256B-I_SP" H 6110 6334 50  0000 C CNN
+F 2 "SeeedOPL-IC-2016:DIP28-2.54-34.7X7.62MM" H 3960 3560 50  0001 C CNN
+F 3 "" H 3960 3560 50  0001 C CNN
+	1    3960 3560
+	1    0    0    -1
+$EndComp
 $EndSCHEMATC

Commit message: lightning controller
lightining controller allen neopixels af te tekenen +voeding
Parts:
- C1, C2, C3, C4, C5, C6: renamed from C?; footprint (none) -> Capacitor_SMD:C_0603_1608Metric
- R3: renamed from R?; footprint (none) -> Resistor_SMD:R_0603_1608Metric
- Y1: renamed from Y?; footprint (none) -> Crystal:Crystal_HC33-U_Vertical
- con1: renamed from con?; footprint (none) -> Connector:Tag-Connect_TC2030-IDC-FP_2x03_P1.27mm_Vertical
- gave numbers to parts that had none: 1
Connections:
- net labels added: DISPIRQ, NEOPIX_OUT1, ~IRQ_ESP
- net labels removed: ~IRQ
- no-connect marks 4 -> 3
Changed lines of the file:
@@
 $Descr A4 11693 8268
 encoding utf-8
-Sheet 2 4
+Sheet 2 5
 Title ""
 Date "2018-10-27"
@@
 	3760 1860 3220 1860
 $Comp
-L power:GND #PWR?
+L power:GND #PWR0103
 U 1 1 5BC88406
 P 3760 2760
-F 0 "#PWR?" H 3760 2510 50  0001 C CNN
+F 0 "#PWR0103" H 3760 2510 50  0001 C CNN
 F 1 "GND" V 3765 2632 50  0000 R CNN
 F 2 "" H 3760 2760 50  0001 C CNN
@@
 PGEC1
 $Comp
-L conectors:icsp con?
+L conectors:icsp con1
 U 1 1 5BC8829D
 P 1160 4220
-F 0 "con?" H 1329 4485 50  0000 C CNN
+F 0 "con1" H 1329 4485 50  0000 C CNN
 F 1 "icsp" H 1329 4394 50  0000 C CNN
-F 2 "" H 1160 4220 50  0001 C CNN
+F 2 "Connector:Tag-Connect_TC2030-IDC-FP_2x03_P1.27mm_Vertical" H 1160 4220 50  0001 C CNN
 F 3 "" H 1160 4220 50  0001 C CNN
 	1    1160 4220
@@
 $EndComp
 $Comp
-L Device:Crystal Y?
+L Device:Crystal Y1
 U 1 1 5BC888B7
 P 1480 2440
-F 0 "Y?" V 1434 2571 50  0000 L CNN
+F 0 "Y1" V 1434 2571 50  0000 L CNN
 F 1 "Crystal" V 1525 2571 50  0000 L CNN
-F 2 "" H 1480 2440 50  0001 C CNN
+F 2 "Crystal:Crystal_HC33-U_Vertical" H 1480 2440 50  0001 C CNN
 F 3 "~" H 1480 2440 50  0001 C CNN
 	1    1480 2440
@@
 $EndComp
 $Comp
-L Device:C_Small C?
+L Device:C_Small C1
 U 1 1 5BC89369
 P 1480 2900
-F 0 "C?" H 1572 2946 50  0000 L CNN
+F 0 "C1" H 1572 2946 50  0000 L CNN
 F 1 "C_Small" H 1572 2855 50  0000 L CNN
-F 2 "" H 1480 2900 50  0001 C CNN
+F 2 "Capacitor_SMD:C_0603_1608Metric" H 1480 2900 50  0001 C CNN
 F 3 "~" H 1480 2900 50  0001 C CNN
 	1    1480 2900
@@
 $EndComp
 $Comp
-L Device:C_Small C?
+L Device:C_Small C2
 U 1 1 5BC8942F
 P 2370 2260
-F 0 "C?" H 2278 2214 50  0000 R CNN
+F 0 "C2" H 2278 2214 50  0000 R CNN
 F 1 "C_Small" H 2278 2305 50  0000 R CNN
-F 2 "" H 2370 2260 50  0001 C CNN
+F 2 "Capacitor_SMD:C_0603_1608Metric" H 2370 2260 50  0001 C CNN
 F 3 "~" H 2370 2260 50  0001 C CNN
 	1    2370 2260
@@
 	1480 2670 1480 2590
 $Comp
-L power:GND #PWR?
+L power:GND #PWR0104
 U 1 1 5BC897F1
 P 1480 3000
-F 0 "#PWR?" H 1480 2750 50  0001 C CNN
+F 0 "#PWR0104" H 1480 2750 50  0001 C CNN
 F 1 "GND" H 1485 2827 50  0000 C CNN
 F 2 "" H 1480 3000 50  0001 C CNN
@@
 $EndComp
 $Comp
-L power:GND #PWR?
+L power:GND #PWR0105
 U 1 1 5BC89810
 P 2370 2360
-F 0 "#PWR?" H 2370 2110 50  0001 C CNN
+F 0 "#PWR0105" H 2370 2110 50  0001 C CNN
 F 1 "GND" H 2375 2187 50  0000 C CNN
 F 2 "" H 2370 2360 50  0001 C CNN
@@
 $EndComp
 $Comp
-L power:GND #PWR?
+L power:GND #PWR0106
 U 1 1 5BC8985C
 P 2610 4460
-F 0 "#PWR?" H 2610 4210 50  0001 C CNN
+F 0 "#PWR0106" H 2610 4210 50  0001 C CNN
 F 1 "GND" H 2615 4287 50  0000 C CNN
 F 2 "" H 2610 4460 50  0001 C CNN
@@
 	1990 4420 1990 4760
 $Comp
-L Device:C_Small C?
+L Device:C_Small C3
 U 1 1 5BC8A895
 P 2610 4360
-F 0 "C?" H 2702 4406 50  0000 L CNN
+F 0 "C3" H 2702 4406 50  0000 L CNN
 F 1 "C_Small" H 2702 4315 50  0000 L CNN
-F 2 "" H 2610 4360 50  0001 C CNN
+F 2 "Capacitor_SMD:C_0603_1608Metric" H 2610 4360 50  0001 C CNN
 F 3 "~" H 2610 4360 50  0001 C CNN
 	1    2610 4360
@@
 $EndComp
 $Comp
-L Device:R R?
+L Device:R R3
 U 1 1 5BC8A9B6
 P 2610 3900
-F 0 "R?" H 2680 3946 50  0000 L CNN
+F 0 "R3" H 2680 3946 50  0000 L CNN
 F 1 "R" H 2680 3855 50  0000 L CNN
-F 2 "" V 2540 3900 50  0001 C CNN
+F 2 "Resistor_SMD:R_0603_1608Metric" V 2540 3900 50  0001 C CNN
 F 3 "~" H 2610 3900 50  0001 C CNN
 	1    2610 3900
@@
 $EndComp
 $Comp
-L power:+3V3 #PWR?
+L power:+3V3 #PWR0107
 U 1 1 5BC8AA4D
 P 2610 3650
-F 0 "#PWR?" H 2610 3500 50  0001 C CNN
+F 0 "#PWR0107" H 2610 3500 50  0001 C CNN
 F 1 "+3V3" H 2625 3823 50  0000 C CNN
 F 2 "" H 2610 3650 50  0001 C CNN
@@
 $EndComp
 $Comp
-L power:+3V3 #PWR?
+L power:+3V3 #PWR0108
 U 1 1 5BC8B3CD
 P 1360 4320
-F 0 "#PWR?" H 1360 4170 50  0001 C CNN
+F 0 "#PWR0108" H 1360 4170 50  0001 C CNN
 F 1 "+3V3" V 1375 4448 50  0000 L CNN
 F 2 "" H 1360 4320 50  0001 C CNN
@@
 	2610 3750 2610 3650
 $Comp
-L power:GND #PWR?
+L power:GND #PWR0109
 U 1 1 5BC8C006
 P 1990 4760
-F 0 "#PWR?" H 1990 4510 50  0001 C CNN
+F 0 "#PWR0109" H 1990 4510 50  0001 C CNN
 F 1 "GND" H 1995 4587 50  0000 C CNN
 F 2 "" H 1990 4760 50  0001 C CNN
@@
 PGEC1
 $Comp
-L power:+3V3 #PWR?
+L power:+3V3 #PWR0110
 U 1 1 5BC8C2BA
 P 3760 2010
-F 0 "#PWR?" H 3760 1860 50  0001 C CNN
+F 0 "#PWR0110" H 3760 1860 50  0001 C CNN
 F 1 "+3V3" V 3775 2138 50  0000 L CNN
 F 2 "" H 3760 2010 50  0001 C CNN
@@
 $EndComp
 $Comp
-L power:+3V3 #PWR?
+L power:+3V3 #PWR0111
 U 1 1 5BC8C304
 P 8460 1160
-F 0 "#PWR?" H 8460 1010 50  0001 C CNN
+F 0 "#PWR0111" H 8460 1010 50  0001 C CNN
 F 1 "+3V3" V 8475 1288 50  0000 L CNN
 F 2 "" H 8460 1160 50  0001 C CNN
@@
 $EndComp
 $Comp
-L power:GND #PWR?
+L power:GND #PWR0112
 U 1 1 5BC8C47C
 P 8460 1010
-F 0 "#PWR?" H 8460 760 50  0001 C CNN
+F 0 "#PWR0112" H 8460 760 50  0001 C CNN
 F 1 "GND" V 8465 882 50  0000 R CNN
 F 2 "" H 8460 1010 50  0001 C CNN
@@
 $EndComp
 $Comp
-L Device:C_Small C?
+L Device:C_Small C6
 U 1 1 5BC8C5E0
 P 9010 2210
-F 0 "C?" V 8781 2210 50  0000 C CNN
-F 1 "C_Small" V 8872 2210 50  0000 C CNN
-F 2 "" H 9010 2210 50  0001 C CNN
+F 0 "C6" V 9060 2290 50  0000 C CNN
+F 1 "C_Small" V 9150 2250 50  0000 C CNN
+F 2 "Capacitor_SMD:C_0603_1608Metric" H 9010 2210 50  0001 C CNN
 F 3 "~" H 9010 2210 50  0001 C CNN
 	1    9010 2210
@@
 	8460 2210 8910 2210
 $Comp
-L power:GND #PWR?
+L power:GND #PWR0113
 U 1 1 5BC8C8F6
 P 9780 2270
-F 0 "#PWR?" H 9780 2020 50  0001 C CNN
+F 0 "#PWR0113" H 9780 2020 50  0001 C CNN
 F 1 "GND" H 9785 2097 50  0000 C CNN
 F 2 "" H 9780 2270 50  0001 C CNN
@@
 	9780 2210 9110 2210
 $Comp
-L power:+3V3 #PWR?
+L power:+3V3 #PWR0114
 U 1 1 5BC8CBE9
 P 8460 2360
-F 0 "#PWR?" H 8460 2210 50  0001 C CNN
+F 0 "#PWR0114" H 8460 2210 50  0001 C CNN
 F 1 "+3V3" V 8475 2488 50  0000 L CNN
 F 2 "" H 8460 2360 50  0001 C CNN
@@
 $EndComp
 $Comp
-L power:+3V3 #PWR?
+L power:+3V3 #PWR0115
 U 1 1 5BC8CECC
 P 2970 5040
-F 0 "#PWR?" H 2970 4890 50  0001 C CNN
+F 0 "#PWR0115" H 2970 4890 50  0001 C CNN
 F 1 "+3V3" H 2985 5213 50  0000 C CNN
 F 2 "" H 2970 5040 50  0001 C CNN
@@
 $EndComp
 $Comp
-L Device:C_Small C?
+L Device:C_Small C5
 U 1 1 5BC8CEE7
 P 3070 5270
-F 0 "C?" H 3162 5270 50  0000 L CNN
+F 0 "C5" H 3162 5270 50  0000 L CNN
 F 1 "C_Small" H 3162 5225 50  0001 L CNN
-F 2 "" H 3070 5270 50  0001 C CNN
+F 2 "Capacitor_SMD:C_0603_1608Metric" H 3070 5270 50  0001 C CNN
 F 3 "~" H 3070 5270 50  0001 C CNN
 	1    3070 5270
@@
 $EndComp
 $Comp
-L Device:C_Small C?
+L Device:C_Small C4
 U 1 1 5BC8CF7B
 P 2870 5280
-F 0 "C?" H 3030 5270 50  0000 R CNN
+F 0 "C4" H 3030 5270 50  0000 R CNN
 F 1 "C_Small" H 2778 5235 50  0001 R CNN
-F 2 "" H 2870 5280 50  0001 C CNN
+F 2 "Capacitor_SMD:C_0603_1608Metric" H 2870 5280 50  0001 C CNN
 F 3 "~" H 2870 5280 50  0001 C CNN
 	1    2870 5280
@@
 	2970 5040 3070 5040
 $Comp
-L power:GND #PWR?
+L power:GND #PWR0116
 U 1 1 5BC8E9CD
 P 2970 5620
-F 0 "#PWR?" H 2970 5370 50  0001 C CNN
+F 0 "#PWR0116" H 2970 5370 50  0001 C CNN
 F 1 "GND" H 2975 5447 50  0000 C CNN
 F 2 "" H 2970 5620 50  0001 C CNN
@@
 NoConn ~ 3760 1110
 NoConn ~ 3760 1260
-NoConn ~ 3760 2910
 NoConn ~ 4780 -15560
 Text Notes 4040 660  0    50   ~ 0
@@
 Text HLabel 8460 1910 2    50   Input ~ 0
 GPIO0
-Text Notes 2990 -470 0    50   ~ 0
-TX en RX op aparte I2C to uart chip\n
 Wire Wire Line
 	3760 2460 3570 2460
 Text HLabel 3570 2460 0    50   Input ~ 0
-~IRQ
+~IRQ_ESP
 Wire Wire Line
 	3760 2610 3550 2610
@@
 RESET
 $Comp
-L Halfgelijders:PIC32MX170F256B-I_SP U?
+L Halfgelijders:PIC32MX170F256B-I_SP U1
 U 1 1 5BC35CAF
 P 3960 3560
-F 0 "U?" H 6110 6425 50  0000 C CNN
+F 0 "U1" H 6110 6425 50  0000 C CNN
 F 1 "PIC32MX170F256B-I_SP" H 6110 6334 50  0000 C CNN
 F 2 "SeeedOPL-IC-2016:DIP28-2.54-34.7X7.62MM" H 3960 3560 50  0001 C CNN
@@
 	1    0    0    -1
 $EndComp
+Text HLabel 8460 2060 2    50   Input ~ 0
+NEOPIX_OUT1
+Text HLabel 8460 2510 2    50   Input ~ 0
+DISPIRQ
 $EndSCHEMATC

Commit message: 7833
voeding en  neopixls verbeterd
Parts:
- con1: footprint Connector:Tag-Connect_TC2030-IDC-FP_2x03_P1.27mm_Vertical -> Connector_IDC:IDC-Header_2x04_P2.54mm_Vertical
Connections:
- net labels removed: DISPIRQ
Changed lines of the file:
@@
 F 0 "con1" H 1329 4485 50  0000 C CNN
 F 1 "icsp" H 1329 4394 50  0000 C CNN
-F 2 "Connector:Tag-Connect_TC2030-IDC-FP_2x03_P1.27mm_Vertical" H 1160 4220 50  0001 C CNN
+F 2 "Connector_IDC:IDC-Header_2x04_P2.54mm_Vertical" H 1160 4220 50  0001 C CNN
 F 3 "" H 1160 4220 50  0001 C CNN
 	1    1160 4220
@@
 Text HLabel 8460 2060 2    50   Input ~ 0
 NEOPIX_OUT1
-Text HLabel 8460 2510 2    50   Input ~ 0
-DISPIRQ
 $EndSCHEMATC

Commit message: 3de bodys toegevoed
pcb 3d view body;s toegevoegd
Parts:
- Y1: footprint Crystal:Crystal_HC33-U_Vertical -> Crystal:Crystal_HC49-U_Horizontal
- con1: footprint Connector_IDC:IDC-Header_2x04_P2.54mm_Vertical -> Connector:Tag-Connect_TC2030-IDC-FP_2x03_P1.27mm_Vertical
Connections:
- no-connect marks 3 -> 8
Changed lines of the file:
@@
 F 0 "con1" H 1329 4485 50  0000 C CNN
 F 1 "icsp" H 1329 4394 50  0000 C CNN
-F 2 "Connector_IDC:IDC-Header_2x04_P2.54mm_Vertical" H 1160 4220 50  0001 C CNN
+F 2 "Connector:Tag-Connect_TC2030-IDC-FP_2x03_P1.27mm_Vertical" H 1160 4220 50  0001 C CNN
 F 3 "" H 1160 4220 50  0001 C CNN
 	1    1160 4220
@@
 F 0 "Y1" V 1434 2571 50  0000 L CNN
 F 1 "Crystal" V 1525 2571 50  0000 L CNN
-F 2 "Crystal:Crystal_HC33-U_Vertical" H 1480 2440 50  0001 C CNN
+F 2 "Crystal:Crystal_HC49-U_Horizontal" H 1480 2440 50  0001 C CNN
 F 3 "~" H 1480 2440 50  0001 C CNN
 	1    1480 2440
@@
 Text HLabel 8460 2060 2    50   Input ~ 0
 NEOPIX_OUT1
+NoConn ~ 3760 2910
+NoConn ~ 8460 2510
+NoConn ~ 8460 2660
+NoConn ~ 8460 2810
+NoConn ~ 8460 2960
 $EndSCHEMATC

Commit message: pic
pic controller en co gerouted
Parts:
- Y1: footprint Crystal:Crystal_HC49-U_Horizontal -> Crystal:Crystal_HC49-4H_Vertical
Changed lines of the file:
@@
 F 0 "Y1" V 1434 2571 50  0000 L CNN
 F 1 "Crystal" V 1525 2571 50  0000 L CNN
-F 2 "Crystal:Crystal_HC49-U_Horizontal" H 1480 2440 50  0001 C CNN
+F 2 "Crystal:Crystal_HC49-4H_Vertical" H 1480 2440 50  0001 C CNN
 F 3 "~" H 1480 2440 50  0001 C CNN
 	1    1480 2440
