File: pcb files/lightnincontroller pcb/lightnincontroller pcb.sch (KiCad schematic (older format))
At the start: 0 parts

Commit message: schemerdetectie
schemerdetectie toegevoegd
Parts:
- added R?: R_PHOTO, symbol Device:R_PHOTO
- added R?: R, symbol Device:R
Connections:
- net labels added: +3.3V, GND
- wire segments 0 -> 5
Other:
- note added: "RX en TX op speciaale I2c to UART chip\n"
Changed lines of the file:
@@
 Comment4 ""
 $EndDescr
+Text Notes 4250 1620 0    50   Italic 10
+RX en TX op speciaale I2c to UART chip\n
 $Sheet
-S 4310 1610 1230 990
+S 3960 2080 1400 2280
 U 5BA79AAB
-F0 "controller" 50
-F1 "controller.sch" 50
+F0 "Sheet5BA79AAB" 0
+F1 "controller.sch" 0
+F2 "SCL" I L 3960 2190 50
+F3 "SDA" I L 3960 2270 50
+F4 "PhotoCel" I L 3960 3700 50
+F5 "CH_PD" I L 3960 2360 50
+F6 "GPIO2" I L 3960 2430 50
+F7 "RST" I L 3960 2500 50
+F8 "GPIO0" I L 3960 2580 50
 $EndSheet
+$Comp
+L power:+3.3V #PWR?
+U 1 1 5BCBD375
+P 3310 3200
+F 0 "#PWR?" H 3310 3050 50  0001 C CNN
+F 1 "+3.3V" H 3325 3373 50  0000 C CNN
+F 2 "" H 3310 3200 50  0001 C CNN
+F 3 "" H 3310 3200 50  0001 C CNN
+	1    3310 3200
+	1    0    0    -1
+$EndComp
+$Comp
+L Device:R_PHOTO R?
+U 1 1 5BCBD424
+P 3310 3500
+F 0 "R?" H 3380 3546 50  0000 L CNN
+F 1 "R_PHOTO" H 3380 3455 50  0000 L CNN
+F 2 "" V 3360 3250 50  0001 L CNN
+F 3 "~" H 3310 3450 50  0001 C CNN
+	1    3310 3500
+	1    0    0    -1
+$EndComp
+$Comp
+L Device:R R?
+U 1 1 5BCBD636
+P 3310 4180
+F 0 "R?" H 3380 4226 50  0000 L CNN
+F 1 "R" H 3380 4135 50  0000 L CNN
+F 2 "" V 3240 4180 50  0001 C CNN
+F 3 "~" H 3310 4180 50  0001 C CNN
+	1    3310 4180
+	1    0    0    -1
+$EndComp
+$Comp
+L power:GND #PWR?
+U 1 1 5BCBD740
+P 3310 4600
+F 0 "#PWR?" H 3310 4350 50  0001 C CNN
+F 1 "GND" H 3315 4427 50  0000 C CNN
+F 2 "" H 3310 4600 50  0001 C CNN
+F 3 "" H 3310 4600 50  0001 C CNN
+	1    3310 4600
+	1    0    0    -1
+$EndComp
+Wire Wire Line
+	3310 4600 3310 4330
+Wire Wire Line
+	3310 3350 3310 3200
+Wire Wire Line
+	3960 3700 3310 3700
+Wire Wire Line
+	3310 3650 3310 3700
+Connection ~ 3310 3700
+Wire Wire Line
+	3310 3700 3310 4030
 $EndSCHEMATC

Commit message: esp en ds1307
gestart aan ds1307 interface
Connections:
- wire segments 5 -> 29
Changed lines of the file:
@@
 $Descr A4 11693 8268
 encoding utf-8
-Sheet 1 2
-Title ""
-Date ""
-Rev ""
+Sheet 1 4
+Title "TOP"
+Date "2018-10-27"
+Rev "V0"
 Comp ""
 Comment1 ""
@@
 U 5BA79AAB
 F0 "Sheet5BA79AAB" 0
-F1 "controller.sch" 0
+F1 "controller.sch" 79
 F2 "SCL" I L 3960 2190 50
-F3 "SDA" I L 3960 2270 50
+F3 "SDA" I L 3960 2260 50
 F4 "PhotoCel" I L 3960 3700 50
-F5 "CH_PD" I L 3960 2360 50
-F6 "GPIO2" I L 3960 2430 50
+F5 "CH_PD" I L 3960 2660 50
+F6 "GPIO2" I L 3960 2580 50
 F7 "RST" I L 3960 2500 50
-F8 "GPIO0" I L 3960 2580 50
+F8 "GPIO0" I L 3960 2750 50
+F9 "~IRQ" I L 3960 2340 50
+F10 "RESET" I L 3960 2420 50
 $EndSheet
 $Comp
@@
 Wire Wire Line
 	3310 3700 3310 4030
+$Sheet
+S 760  2090 1420 700
+U 5BCCFC94
+F0 "Sheet5BCCFC93" 0
+F1 "ESP8266.sch" 50
+F2 "GPIO_0" I R 2180 2720 50
+F3 "RTS" I R 2180 2470 50
+F4 "GPIO2" I R 2180 2550 50
+F5 "CH_PD" I R 2180 2650 50
+F6 "~IRQ" I R 2180 2300 50
+F7 "SCL" I R 2180 2150 50
+F8 "SDA" I R 2180 2220 50
+F9 "RESET" I R 2180 2380 50
+$EndSheet
+Wire Wire Line
+	2180 2150 3920 2150
+Wire Wire Line
+	3920 2150 3920 2190
+Wire Wire Line
+	3920 2190 3960 2190
+Wire Wire Line
+	2180 2300 3690 2300
+Wire Wire Line
+	3690 2300 3690 2340
+Wire Wire Line
+	3690 2340 3960 2340
+Wire Wire Line
+	3960 2420 3130 2420
+Wire Wire Line
+	3130 2420 3130 2380
+Wire Wire Line
+	3130 2380 2180 2380
+Wire Wire Line
+	3860 2470 3860 2500
+Wire Wire Line
+	3860 2500 3960 2500
+Wire Wire Line
+	2180 2470 3860 2470
+Wire Wire Line
+	3960 2580 3130 2580
+Wire Wire Line
+	3130 2580 3130 2550
+Wire Wire Line
+	3130 2550 2180 2550
+Wire Wire Line
+	3940 2650 3940 2660
+Wire Wire Line
+	3940 2660 3960 2660
+Wire Wire Line
+	2300 2750 2300 2720
+Wire Wire Line
+	2300 2720 2180 2720
+Wire Wire Line
+	2300 2750 3960 2750
+Wire Wire Line
+	2180 2220 3910 2220
+Wire Wire Line
+	3910 2220 3910 2260
+Wire Wire Line
+	3910 2260 3960 2260
+Wire Wire Line
+	2180 2650 3940 2650
+$Sheet
+S 840  1120 1260 850
+U 5BD55925
+F0 "Sheet5BD55924" 0
+F1 "RTC.sch" 50
+$EndSheet
 $EndSCHEMATC

Commit message: RTC
RTC afgetekend
Connections:
- wire segments 29 -> 35
Other:
- note removed: "RX en TX op speciaale I2c to UART chip\n"
Changed lines of the file:
@@
 Comment4 ""
 $EndDescr
-Text Notes 4250 1620 0    50   Italic 10
-RX en TX op speciaale I2c to UART chip\n
 $Sheet
 S 3960 2080 1400 2280
@@
 $EndSheet
 Wire Wire Line
-	2180 2150 3920 2150
+	2180 2150 2380 2150
 Wire Wire Line
 	3920 2150 3920 2190
@@
 	2300 2750 3960 2750
 Wire Wire Line
-	2180 2220 3910 2220
-Wire Wire Line
 	3910 2220 3910 2260
 Wire Wire Line
@@
 	2180 2650 3940 2650
 $Sheet
-S 840  1120 1260 850
+S 1090 1280 510  540
 U 5BD55925
 F0 "Sheet5BD55924" 0
 F1 "RTC.sch" 50
+F2 "SCL" I R 1600 1550 50
+F3 "SDA" I R 1600 1640 50
 $EndSheet
+Wire Wire Line
+	2380 1550 2380 2150
+Connection ~ 2380 2150
+Wire Wire Line
+	2380 2150 3920 2150
+Wire Wire Line
+	1600 1550 2380 1550
+Wire Wire Line
+	2180 2220 2300 2220
+Wire Wire Line
+	1600 1640 2300 1640
+Wire Wire Line
+	2300 1640 2300 2220
+Connection ~ 2300 2220
+Wire Wire Line
+	2300 2220 3910 2220
 $EndSCHEMATC

Commit message: lightning controller
lightining controller allen neopixels af te tekenen +voeding
Parts:
- R1: renamed from R?; footprint (none) -> Resistor_THT:R_Axial_Power_L20.0mm_W6.4mm_P7.62mm_Vertical
- R2: renamed from R?; footprint (none) -> Resistor_SMD:R_0603_1608Metric
Connections:
- wire segments 35 -> 37
Changed lines of the file:
@@
 $Descr A4 11693 8268
 encoding utf-8
-Sheet 1 4
+Sheet 1 5
 Title "TOP"
 Date "2018-10-27"
@@
 $EndDescr
 $Sheet
-S 3960 2080 1400 2280
+S 4600 4000 1400 2280
 U 5BA79AAB
 F0 "Sheet5BA79AAB" 0
 F1 "controller.sch" 79
-F2 "SCL" I L 3960 2190 50
-F3 "SDA" I L 3960 2260 50
-F4 "PhotoCel" I L 3960 3700 50
-F5 "CH_PD" I L 3960 2660 50
-F6 "GPIO2" I L 3960 2580 50
-F7 "RST" I L 3960 2500 50
-F8 "GPIO0" I L 3960 2750 50
-F9 "~IRQ" I L 3960 2340 50
-F10 "RESET" I L 3960 2420 50
+F2 "SCL" I L 4600 4110 50
+F3 "SDA" I L 4600 4180 50
+F4 "PhotoCel" I L 4600 5620 50
+F5 "CH_PD" I L 4600 4580 50
+F6 "GPIO2" I L 4600 4500 50
+F7 "RST" I L 4600 4420 50
+F8 "GPIO0" I L 4600 4670 50
+F9 "RESET" I L 4600 4340 50
+F10 "~IRQ_ESP" I L 4600 4260 50
+F11 "NEOPIX_OUT1" I R 6000 5120 50
+F12 "DISPIRQ" I L 4600 4900 50
 $EndSheet
 $Comp
-L power:+3.3V #PWR?
+L power:+3.3V #PWR0101
 U 1 1 5BCBD375
-P 3310 3200
-F 0 "#PWR?" H 3310 3050 50  0001 C CNN
-F 1 "+3.3V" H 3325 3373 50  0000 C CNN
-F 2 "" H 3310 3200 50  0001 C CNN
-F 3 "" H 3310 3200 50  0001 C CNN
-	1    3310 3200
+P 3950 5120
+F 0 "#PWR0101" H 3950 4970 50  0001 C CNN
+F 1 "+3.3V" H 3965 5293 50  0000 C CNN
+F 2 "" H 3950 5120 50  0001 C CNN
+F 3 "" H 3950 5120 50  0001 C CNN
+	1    3950 5120
 	1    0    0    -1
 $EndComp
 $Comp
-L Device:R_PHOTO R?
+L Device:R_PHOTO R1
 U 1 1 5BCBD424
-P 3310 3500
-F 0 "R?" H 3380 3546 50  0000 L CNN
-F 1 "R_PHOTO" H 3380 3455 50  0000 L CNN
-F 2 "" V 3360 3250 50  0001 L CNN
-F 3 "~" H 3310 3450 50  0001 C CNN
-	1    3310 3500
+P 3950 5420
+F 0 "R1" H 4020 5466 50  0000 L CNN
+F 1 "R_PHOTO" H 4020 5375 50  0000 L CNN
+F 2 "Resistor_THT:R_Axial_Power_L20.0mm_W6.4mm_P7.62mm_Vertical" V 4000 5170 50  0001 L CNN
+F 3 "~" H 3950 5370 50  0001 C CNN
+	1    3950 5420
 	1    0    0    -1
 $EndComp
 $Comp
-L Device:R R?
+L Device:R R2
 U 1 1 5BCBD636
-P 3310 4180
-F 0 "R?" H 3380 4226 50  0000 L CNN
-F 1 "R" H 3380 4135 50  0000 L CNN
-F 2 "" V 3240 4180 50  0001 C CNN
-F 3 "~" H 3310 4180 50  0001 C CNN
-	1    3310 4180
+P 3950 6100
+F 0 "R2" H 4020 6146 50  0000 L CNN
+F 1 "R" H 4020 6055 50  0000 L CNN
+F 2 "Resistor_SMD:R_0603_1608Metric" V 3880 6100 50  0001 C CNN
+F 3 "~" H 3950 6100 50  0001 C CNN
+	1    3950 6100
 	1    0    0    -1
 $EndComp
 $Comp
-L power:GND #PWR?
+L power:GND #PWR0102
 U 1 1 5BCBD740
-P 3310 4600
-F 0 "#PWR?" H 3310 4350 50  0001 C CNN
-F 1 "GND" H 3315 4427 50  0000 C CNN
-F 2 "" H 3310 4600 50  0001 C CNN
-F 3 "" H 3310 4600 50  0001 C CNN
-	1    3310 4600
+P 3950 6520
+F 0 "#PWR0102" H 3950 6270 50  0001 C CNN
+F 1 "GND" H 3955 6347 50  0000 C CNN
+F 2 "" H 3950 6520 50  0001 C CNN
+F 3 "" H 3950 6520 50  0001 C CNN
+	1    3950 6520
 	1    0    0    -1
 $EndComp
 Wire Wire Line
-	3310 4600 3310 4330
+	3950 6520 3950 6250
 Wire Wire Line
-	3310 3350 3310 3200
+	3950 5270 3950 5120
 Wire Wire Line
-	3960 3700 3310 3700
+	4600 5620 3950 5620
 Wire Wire Line
-	3310 3650 3310 3700
-Connection ~ 3310 3700
+	3950 5570 3950 5620
+Connection ~ 3950 5620
 Wire Wire Line
-	3310 3700 3310 4030
+	3950 5620 3950 5950
 $Sheet
-S 760  2090 1420 700
+S 1400 4010 1420 700
 U 5BCCFC94
 F0 "Sheet5BCCFC93" 0
 F1 "ESP8266.sch" 50
-F2 "GPIO_0" I R 2180 2720 50
-F3 "RTS" I R 2180 2470 50
-F4 "GPIO2" I R 2180 2550 50
-F5 "CH_PD" I R 2180 2650 50
-F6 "~IRQ" I R 2180 2300 50
-F7 "SCL" I R 2180 2150 50
-F8 "SDA" I R 2180 2220 50
-F9 "RESET" I R 2180 2380 50
+F2 "GPIO_0" I R 2820 4640 50
+F3 "RTS" I R 2820 4390 50
+F4 "GPIO2" I R 2820 4470 50
+F5 "CH_PD" I R 2820 4570 50
+F6 "~IRQ" I R 2820 4220 50
+F7 "SCL" I R 2820 4070 50
+F8 "SDA" I R 2820 4140 50
+F9 "RESET" I R 2820 4300 50
 $EndSheet
 Wire Wire Line
-	2180 2150 2380 2150
+	2820 4070 3020 4070
 Wire Wire Line
-	3920 2150 3920 2190
+	4560 4070 4560 4110
 Wire Wire Line
-	3920 2190 3960 2190
+	4560 4110 4600 4110
 Wire Wire Line
-	2180 2300 3690 2300
+	2820 4220 4330 4220
 Wire Wire Line
-	3690 2300 3690 2340
+	4330 4220 4330 4260
 Wire Wire Line
-	3690 2340 3960 2340
+	4330 4260 4600 4260
 Wire Wire Line
-	3960 2420 3130 2420
+	4600 4340 3770 4340
 Wire Wire Line
-	3130 2420 3130 2380
+	3770 4340 3770 4300
 Wire Wire Line
-	3130 2380 2180 2380
+	3770 4300 2820 4300
 Wire Wire Line
-	3860 2470 3860 2500
+	4500 4390 4500 4420
 Wire Wire Line
-	3860 2500 3960 2500
+	4500 4420 4600 4420
 Wire Wire Line
-	2180 2470 3860 2470
+	2820 4390 4500 4390
 Wire Wire Line
-	3960 2580 3130 2580
+	4600 4500 3770 4500
 Wire Wire Line
-	3130 2580 3130 2550
+	3770 4500 3770 4470
 Wire Wire Line
-	3130 2550 2180 2550
+	3770 4470 2820 4470
 Wire Wire Line
-	3940 2650 3940 2660
+	4580 4570 4580 4580
 Wire Wire Line
-	3940 2660 3960 2660
+	4580 4580 4600 4580
 Wire Wire Line
-	2300 2750 2300 2720
+	2940 4670 2940 4640
 Wire Wire Line
-	2300 2720 2180 2720
+	2940 4640 2820 4640
 Wire Wire Line
-	2300 2750 3960 2750
+	2940 4670 4600 4670
 Wire Wire Line
-	3910 2220 3910 2260
+	4550 4140 4550 4180
 Wire Wire Line
-	3910 2260 3960 2260
+	4550 4180 4600 4180
 Wire Wire Line
-	2180 2650 3940 2650
+	2820 4570 4580 4570
 $Sheet
-S 1090 1280 510  540
+S 1730 3200 510  540
 U 5BD55925
 F0 "Sheet5BD55924" 0
 F1 "RTC.sch" 50
-F2 "SCL" I R 1600 1550 50
-F3 "SDA" I R 1600 1640 50
+F2 "SCL" I R 2240 3470 50
+F3 "SDA" I R 2240 3560 50
 $EndSheet
 Wire Wire Line
-	2380 1550 2380 2150
-Connection ~ 2380 2150
+	3020 3470 3020 4070
+Connection ~ 3020 4070
 Wire Wire Line
-	2380 2150 3920 2150
+	3020 4070 4560 4070
 Wire Wire Line
-	1600 1550 2380 1550
+	2240 3470 3020 3470
 Wire Wire Line
-	2180 2220 2300 2220
+	2820 4140 2940 4140
 Wire Wire Line
-	1600 1640 2300 1640
+	2240 3560 2940 3560
 Wire Wire Line
-	2300 1640 2300 2220
-Connection ~ 2300 2220
+	2940 3560 2940 4140
+Connection ~ 2940 4140
 Wire Wire Line
-	2300 2220 3910 2220
+	2940 4140 4550 4140
+$Sheet
+S 6310 4820 1060 610
+U 5BD4F2FD
+F0 "Sheet5BD4F2FC" 0
+F1 "NEOPIX.sch" 50
+F2 "NEOPIX_in" I L 6310 5110 50
+F3 "NEOPIX_out" I R 7370 5120 50
+$EndSheet
+Wire Wire Line
+	6000 5120 6310 5120
+Wire Wire Line
+	6310 5120 6310 5110
 $EndSCHEMATC

Commit message: neopixel
neopixels ingetekend
Connections:
- wire segments 37 -> 38
Changed lines of the file:
@@
 $Descr A4 11693 8268
 encoding utf-8
-Sheet 1 5
+Sheet 1 6
 Title "TOP"
 Date "2018-10-27"
@@
 $EndDescr
 $Sheet
-S 4600 4000 1400 2280
+S 6830 2530 1400 2280
 U 5BA79AAB
 F0 "Sheet5BA79AAB" 0
 F1 "controller.sch" 79
-F2 "SCL" I L 4600 4110 50
-F3 "SDA" I L 4600 4180 50
-F4 "PhotoCel" I L 4600 5620 50
-F5 "CH_PD" I L 4600 4580 50
-F6 "GPIO2" I L 4600 4500 50
-F7 "RST" I L 4600 4420 50
-F8 "GPIO0" I L 4600 4670 50
-F9 "RESET" I L 4600 4340 50
-F10 "~IRQ_ESP" I L 4600 4260 50
-F11 "NEOPIX_OUT1" I R 6000 5120 50
-F12 "DISPIRQ" I L 4600 4900 50
+F2 "SCL" I L 6830 2640 50
+F3 "SDA" I L 6830 2710 50
+F4 "PhotoCel" I L 6830 4150 50
+F5 "CH_PD" I L 6830 3110 50
+F6 "GPIO2" I L 6830 3030 50
+F7 "RST" I L 6830 2950 50
+F8 "GPIO0" I L 6830 3200 50
+F9 "RESET" I L 6830 2870 50
+F10 "~IRQ_ESP" I L 6830 2790 50
+F11 "NEOPIX_OUT1" I R 8230 3650 50
+F12 "DISPIRQ" I L 6830 3430 50
 $EndSheet
 $Comp
 L power:+3.3V #PWR0101
 U 1 1 5BCBD375
-P 3950 5120
-F 0 "#PWR0101" H 3950 4970 50  0001 C CNN
-F 1 "+3.3V" H 3965 5293 50  0000 C CNN
-F 2 "" H 3950 5120 50  0001 C CNN
-F 3 "" H 3950 5120 50  0001 C CNN
-	1    3950 5120
+P 6180 3650
+F 0 "#PWR0101" H 6180 3500 50  0001 C CNN
+F 1 "+3.3V" H 6195 3823 50  0000 C CNN
+F 2 "" H 6180 3650 50  0001 C CNN
+F 3 "" H 6180 3650 50  0001 C CNN
+	1    6180 3650
 	1    0    0    -1
 $EndComp
@@
 L Device:R_PHOTO R1
 U 1 1 5BCBD424
-P 3950 5420
-F 0 "R1" H 4020 5466 50  0000 L CNN
-F 1 "R_PHOTO" H 4020 5375 50  0000 L CNN
-F 2 "Resistor_THT:R_Axial_Power_L20.0mm_W6.4mm_P7.62mm_Vertical" V 4000 5170 50  0001 L CNN
-F 3 "~" H 3950 5370 50  0001 C CNN
-	1    3950 5420
+P 6180 3950
+F 0 "R1" H 6250 3996 50  0000 L CNN
+F 1 "R_PHOTO" H 6250 3905 50  0000 L CNN
+F 2 "Resistor_THT:R_Axial_Power_L20.0mm_W6.4mm_P7.62mm_Vertical" V 6230 3700 50  0001 L CNN
+F 3 "~" H 6180 3900 50  0001 C CNN
+	1    6180 3950
 	1    0    0    -1
 $EndComp
@@
 L Device:R R2
 U 1 1 5BCBD636
-P 3950 6100
-F 0 "R2" H 4020 6146 50  0000 L CNN
-F 1 "R" H 4020 6055 50  0000 L CNN
-F 2 "Resistor_SMD:R_0603_1608Metric" V 3880 6100 50  0001 C CNN
-F 3 "~" H 3950 6100 50  0001 C CNN
-	1    3950 6100
+P 6180 4630
+F 0 "R2" H 6250 4676 50  0000 L CNN
+F 1 "R" H 6250 4585 50  0000 L CNN
+F 2 "Resistor_SMD:R_0603_1608Metric" V 6110 4630 50  0001 C CNN
+F 3 "~" H 6180 4630 50  0001 C CNN
+	1    6180 4630
 	1    0    0    -1
 $EndComp
@@
 L power:GND #PWR0102
 U 1 1 5BCBD740
-P 3950 6520
-F 0 "#PWR0102" H 3950 6270 50  0001 C CNN
-F 1 "GND" H 3955 6347 50  0000 C CNN
-F 2 "" H 3950 6520 50  0001 C CNN
-F 3 "" H 3950 6520 50  0001 C CNN
-	1    3950 6520
+P 6180 5050
+F 0 "#PWR0102" H 6180 4800 50  0001 C CNN
+F 1 "GND" H 6185 4877 50  0000 C CNN
+F 2 "" H 6180 5050 50  0001 C CNN
+F 3 "" H 6180 5050 50  0001 C CNN
+	1    6180 5050
 	1    0    0    -1
 $EndComp
 Wire Wire Line
-	3950 6520 3950 6250
+	6180 5050 6180 4780
 Wire Wire Line
-	3950 5270 3950 5120
+	6180 3800 6180 3650
 Wire Wire Line
-	4600 5620 3950 5620
+	6830 4150 6180 4150
 Wire Wire Line
-	3950 5570 3950 5620
-Connection ~ 3950 5620
+	6180 4100 6180 4150
+Connection ~ 6180 4150
 Wire Wire Line
-	3950 5620 3950 5950
+	6180 4150 6180 4480
 $Sheet
-S 1400 4010 1420 700
+S 3630 2540 1420 700
 U 5BCCFC94
 F0 "Sheet5BCCFC93" 0
 F1 "ESP8266.sch" 50
-F2 "GPIO_0" I R 2820 4640 50
-F3 "RTS" I R 2820 4390 50
-F4 "GPIO2" I R 2820 4470 50
-F5 "CH_PD" I R 2820 4570 50
-F6 "~IRQ" I R 2820 4220 50
-F7 "SCL" I R 2820 4070 50
-F8 "SDA" I R 2820 4140 50
-F9 "RESET" I R 2820 4300 50
+F2 "GPIO_0" I R 5050 3170 50
+F3 "RTS" I R 5050 2920 50
+F4 "GPIO2" I R 5050 3000 50
+F5 "CH_PD" I R 5050 3100 50
+F6 "~IRQ" I R 5050 2750 50
+F7 "SCL" I R 5050 2600 50
+F8 "SDA" I R 5050 2670 50
+F9 "RESET" I R 5050 2830 50
 $EndSheet
 Wire Wire Line
-	2820 4070 3020 4070
+	5050 2600 5250 2600
 Wire Wire Line
-	4560 4070 4560 4110
+	6790 2600 6790 2640
 Wire Wire Line
-	4560 4110 4600 4110
+	6790 2640 6830 2640
 Wire Wire Line
-	2820 4220 4330 4220
+	5050 2750 6560 2750
 Wire Wire Line
-	4330 4220 4330 4260
+	6560 2750 6560 2790
 Wire Wire Line
-	4330 4260 4600 4260
+	6560 2790 6830 2790
 Wire Wire Line
-	4600 4340 3770 4340
+	6830 2870 6000 2870
 Wire Wire Line
-	3770 4340 3770 4300
+	6000 2870 6000 2830
 Wire Wire Line
-	3770 4300 2820 4300
+	6000 2830 5050 2830
 Wire Wire Line
-	4500 4390 4500 4420
+	6730 2920 6730 2950
 Wire Wire Line
-	4500 4420 4600 4420
+	6730 2950 6830 2950
 Wire Wire Line
-	2820 4390 4500 4390
+	5050 2920 6730 2920
 Wire Wire Line
-	4600 4500 3770 4500
+	6830 3030 6000 3030
 Wire Wire Line
-	3770 4500 3770 4470
+	6000 3030 6000 3000
 Wire Wire Line
-	3770 4470 2820 4470
+	6000 3000 5050 3000
 Wire Wire Line
-	4580 4570 4580 4580
+	6810 3100 6810 3110
 Wire Wire Line
-	4580 4580 4600 4580
+	6810 3110 6830 3110
 Wire Wire Line
-	2940 4670 2940 4640
+	5170 3200 5170 3170
 Wire Wire Line
-	2940 4640 2820 4640
+	5170 3170 5050 3170
 Wire Wire Line
-	2940 4670 4600 4670
+	5170 3200 6830 3200
 Wire Wire Line
-	4550 4140 4550 4180
+	6780 2670 6780 2710
 Wire Wire Line
-	4550 4180 4600 4180
+	6780 2710 6830 2710
 Wire Wire Line
-	2820 4570 4580 4570
+	5050 3100 6810 3100
 $Sheet
-S 1730 3200 510  540
+S 3960 1730 510  540
 U 5BD55925
 F0 "Sheet5BD55924" 0
 F1 "RTC.sch" 50
-F2 "SCL" I R 2240 3470 50
-F3 "SDA" I R 2240 3560 50
+F2 "SCL" I R 4470 2000 50
+F3 "SDA" I R 4470 2090 50
 $EndSheet
 Wire Wire Line
-	3020 3470 3020 4070
-Connection ~ 3020 4070
+	5250 2000 5250 2600
+Connection ~ 5250 2600
 Wire Wire Line
-	3020 4070 4560 4070
+	5250 2600 6790 2600
 Wire Wire Line
-	2240 3470 3020 3470
+	4470 2000 5250 2000
 Wire Wire Line
-	2820 4140 2940 4140
+	5050 2670 5170 2670
 Wire Wire Line
-	2240 3560 2940 3560
+	4470 2090 5170 2090
 Wire Wire Line
-	2940 3560 2940 4140
-Connection ~ 2940 4140
+	5170 2090 5170 2670
+Connection ~ 5170 2670
 Wire Wire Line
-	2940 4140 4550 4140
+	5170 2670 6780 2670
 $Sheet
-S 6310 4820 1060 610
+S 8540 3350 1060 610
 U 5BD4F2FD
 F0 "Sheet5BD4F2FC" 0
 F1 "NEOPIX.sch" 50
-F2 "NEOPIX_in" I L 6310 5110 50
-F3 "NEOPIX_out" I R 7370 5120 50
+F2 "NEOPIX_in" I L 8540 3640 50
+F3 "NEOPIX_out" I R 9600 3650 50
 $EndSheet
 Wire Wire Line
-	6000 5120 6310 5120
+	8230 3650 8540 3650
 Wire Wire Line
-	6310 5120 6310 5110
+	8540 3650 8540 3640
+$Sheet
+S 9740 3330 1000 660
+U 5BFAE0EC
+F0 "Sheet5BFAE0EB" 0
+F1 "Neopixels.sch" 50
+F2 "DI" I L 9740 3650 50
+$EndSheet
+Wire Wire Line
+	9600 3650 9740 3650
 $EndSCHEMATC

Commit message: 7833
voeding en  neopixls verbeterd
Connections:
- wire segments 38 -> 32
Changed lines of the file:
@@
 S 6830 2530 1400 2280
 U 5BA79AAB
-F0 "Sheet5BA79AAB" 0
+F0 "controller" 79
 F1 "controller.sch" 79
 F2 "SCL" I L 6830 2640 50
@@
 S 3630 2540 1420 700
 U 5BCCFC94
-F0 "Sheet5BCCFC93" 0
+F0 "ESP8266" 50
 F1 "ESP8266.sch" 50
 F2 "GPIO_0" I R 5050 3170 50
@@
 F9 "RESET" I R 5050 2830 50
 $EndSheet
-Wire Wire Line
-	5050 2600 5250 2600
 Wire Wire Line
 	6790 2600 6790 2640
@@
 	5050 3100 6810 3100
 $Sheet
-S 3960 1730 510  540
-U 5BD55925
-F0 "Sheet5BD55924" 0
-F1 "RTC.sch" 50
-F2 "SCL" I R 4470 2000 50
-F3 "SDA" I R 4470 2090 50
-$EndSheet
-Wire Wire Line
-	5250 2000 5250 2600
-Connection ~ 5250 2600
-Wire Wire Line
-	5250 2600 6790 2600
-Wire Wire Line
-	4470 2000 5250 2000
-Wire Wire Line
-	5050 2670 5170 2670
-Wire Wire Line
-	4470 2090 5170 2090
-Wire Wire Line
-	5170 2090 5170 2670
-Connection ~ 5170 2670
-Wire Wire Line
-	5170 2670 6780 2670
-$Sheet
 S 8540 3350 1060 610
 U 5BD4F2FD
-F0 "Sheet5BD4F2FC" 0
+F0 "NEOPIX" 50
 F1 "NEOPIX.sch" 50
 F2 "NEOPIX_in" I L 8540 3640 50
@@
 Wire Wire Line
 	9600 3650 9740 3650
+Wire Wire Line
+	5050 2600 6790 2600
+Wire Wire Line
+	5050 2670 6780 2670
+$Sheet
+S 1620 2730 720  440
+U 5C1941A3
+F0 "voeding " 50
+F1 "voeding.sch" 50
+$EndSheet
 $EndSCHEMATC

Commit message: 3de bodys toegevoed
pcb 3d view body;s toegevoegd
Other:
- note added: "\nTO-DO\nComponnenten waardes geven"
Changed lines of the file:
@@
 F10 "~IRQ_ESP" I L 6830 2790 50
 F11 "NEOPIX_OUT1" I R 8230 3650 50
-F12 "DISPIRQ" I L 6830 3430 50
 $EndSheet
 $Comp
@@
 S 9740 3330 1000 660
 U 5BFAE0EC
-F0 "Sheet5BFAE0EB" 0
+F0 "Neopixel" 50
 F1 "Neopixels.sch" 50
 F2 "DI" I L 9740 3650 50
@@
 	5050 2670 6780 2670
 $Sheet
-S 1620 2730 720  440
+S 7460 5500 3270 910
 U 5C1941A3
 F0 "voeding " 50
 F1 "voeding.sch" 50
 $EndSheet
+Wire Notes Line
+	8150 5500 8150 4810
+Wire Notes Line
+	8150 4810 8090 4870
+Wire Notes Line
+	8150 4810 8210 4870
+Wire Notes Line
+	10600 5500 10590 4010
+Wire Notes Line
+	10590 4010 10560 4050
+Wire Notes Line
+	10590 4010 10620 4050
+Text Notes 5790 1490 0    197  Italic 39
+\nTO-DO\nComponnenten waardes geven
 $EndSCHEMATC

Commit message: pic
pic controller en co gerouted
Parts:
- R1: footprint Resistor_THT:R_Axial_Power_L20.0mm_W6.4mm_P7.62mm_Vertical -> Resistor_THT:R_Axial_DIN0204_L3.6mm_D1.6mm_P1.90mm_Vertical
Changed lines of the file:
@@
 F 0 "R1" H 6250 3996 50  0000 L CNN
 F 1 "R_PHOTO" H 6250 3905 50  0000 L CNN
-F 2 "Resistor_THT:R_Axial_Power_L20.0mm_W6.4mm_P7.62mm_Vertical" V 6230 3700 50  0001 L CNN
+F 2 "Resistor_THT:R_Axial_DIN0204_L3.6mm_D1.6mm_P1.90mm_Vertical" V 6230 3700 50  0001 L CNN
 F 3 "~" H 6180 3900 50  0001 C CNN
 	1    6180 3950
