File: pcb files/lightnincontroller pcb/voeding.sch (KiCad schematic (older format))
At the start: 1 part, among them J1 Screw_Terminal_01x02

Commit message: 3de bodys toegevoed
pcb 3d view body;s toegevoegd
Parts:
- added C14, C15, C16, C19: C_Small, Capacitor_SMD:C_0603_1608Metric, symbol Device:C_Small
- added C20: C_Small, Capacitor_THT:CP_Radial_D10.0mm_P2.50mm_P5.00mm, symbol Device:C_Small
- added U3: 7833, Package_TO_SOT_THT:TO-220-3_Vertical, symbol Halfgelijders:7833
Connections:
- net labels added: +3V3, GND, VCC
- wire segments 0 -> 21
Changed lines of the file:
@@
 	-1   0    0    1
 $EndComp
+$Comp
+L Halfgelijders:7833 U3
+U 1 1 5C1F8A10
+P 3640 3050
+F 0 "U3" H 3890 3465 50  0000 C CNN
+F 1 "7833" H 3890 3374 50  0000 C CNN
+F 2 "Package_TO_SOT_THT:TO-220-3_Vertical" H 3640 3050 50  0001 C CNN
+F 3 "" H 3640 3050 50  0001 C CNN
+	1    3640 3050
+	1    0    0    -1
+$EndComp
+Wire Wire Line
+	2510 3000 2880 3000
+$Comp
+L power:VCC #PWR05
+U 1 1 5C1FB985
+P 2880 3000
+F 0 "#PWR05" H 2880 2850 50  0001 C CNN
+F 1 "VCC" H 2897 3173 50  0000 C CNN
+F 2 "" H 2880 3000 50  0001 C CNN
+F 3 "" H 2880 3000 50  0001 C CNN
+	1    2880 3000
+	1    0    0    -1
+$EndComp
+Connection ~ 2880 3000
+Wire Wire Line
+	2880 3000 3440 3000
+Wire Wire Line
+	2510 3100 2880 3100
+Wire Wire Line
+	2880 3100 2880 3340
+$Comp
+L power:GND #PWR09
+U 1 1 5C1FBA12
+P 3890 3300
+F 0 "#PWR09" H 3890 3050 50  0001 C CNN
+F 1 "GND" H 3895 3127 50  0000 C CNN
+F 2 "" H 3890 3300 50  0001 C CNN
+F 3 "" H 3890 3300 50  0001 C CNN
+	1    3890 3300
+	1    0    0    -1
+$EndComp
+$Comp
+L power:GND #PWR06
+U 1 1 5C1FBA28
+P 2880 3340
+F 0 "#PWR06" H 2880 3090 50  0001 C CNN
+F 1 "GND" H 2885 3167 50  0000 C CNN
+F 2 "" H 2880 3340 50  0001 C CNN
+F 3 "" H 2880 3340 50  0001 C CNN
+	1    2880 3340
+	1    0    0    -1
+$EndComp
+Wire Wire Line
+	4340 3000 4950 3000
+$Comp
+L power:+3V3 #PWR010
+U 1 1 5C1FBA81
+P 4950 3000
+F 0 "#PWR010" H 4950 2850 50  0001 C CNN
+F 1 "+3V3" H 4965 3173 50  0000 C CNN
+F 2 "" H 4950 3000 50  0001 C CNN
+F 3 "" H 4950 3000 50  0001 C CNN
+	1    4950 3000
+	1    0    0    -1
+$EndComp
+$Comp
+L Device:C_Small C14
+U 1 1 5C1FBC5C
+P 2430 4900
+F 0 "C14" H 2338 4854 50  0000 R CNN
+F 1 "C_Small" H 2338 4945 50  0000 R CNN
+F 2 "Capacitor_SMD:C_0603_1608Metric" H 2430 4900 50  0001 C CNN
+F 3 "~" H 2430 4900 50  0001 C CNN
+	1    2430 4900
+	1    0    0    1
+$EndComp
+$Comp
+L Device:C_Small C15
+U 1 1 5C1FBCC3
+P 2630 4900
+F 0 "C15" H 2722 4946 50  0000 L CNN
+F 1 "C_Small" H 2722 4855 50  0000 L CNN
+F 2 "Capacitor_SMD:C_0603_1608Metric" H 2630 4900 50  0001 C CNN
+F 3 "~" H 2630 4900 50  0001 C CNN
+	1    2630 4900
+	1    0    0    -1
+$EndComp
+$Comp
+L power:GND #PWR04
+U 1 1 5C1FBDB0
+P 2520 5060
+F 0 "#PWR04" H 2520 4810 50  0001 C CNN
+F 1 "GND" H 2525 4887 50  0000 C CNN
+F 2 "" H 2520 5060 50  0001 C CNN
+F 3 "" H 2520 5060 50  0001 C CNN
+	1    2520 5060
+	1    0    0    -1
+$EndComp
+$Comp
+L power:VCC #PWR03
+U 1 1 5C1FBDC3
+P 2520 4690
+F 0 "#PWR03" H 2520 4540 50  0001 C CNN
+F 1 "VCC" H 2537 4863 50  0000 C CNN
+F 2 "" H 2520 4690 50  0001 C CNN
+F 3 "" H 2520 4690 50  0001 C CNN
+	1    2520 4690
+	1    0    0    -1
+$EndComp
+$Comp
+L Device:C_Small C16
+U 1 1 5C1FBDD6
+P 3680 4950
+F 0 "C16" H 3588 4904 50  0000 R CNN
+F 1 "C_Small" H 3588 4995 50  0000 R CNN
+F 2 "Capacitor_SMD:C_0603_1608Metric" H 3680 4950 50  0001 C CNN
+F 3 "~" H 3680 4950 50  0001 C CNN
+	1    3680 4950
+	1    0    0    1
+$EndComp
+$Comp
+L Device:C_Small C19
+U 1 1 5C1FBE32
+P 3930 4940
+F 0 "C19" H 4022 4986 50  0000 L CNN
+F 1 "C_Small" H 4022 4895 50  0000 L CNN
+F 2 "Capacitor_SMD:C_0603_1608Metric" H 3930 4940 50  0001 C CNN
+F 3 "~" H 3930 4940 50  0001 C CNN
+	1    3930 4940
+	1    0    0    -1
+$EndComp
+Wire Wire Line
+	2430 4800 2430 4690
+Wire Wire Line
+	2430 4690 2520 4690
+Wire Wire Line
+	2630 4690 2630 4800
+Connection ~ 2520 4690
+Wire Wire Line
+	2520 4690 2630 4690
+Wire Wire Line
+	2430 5000 2430 5060
+Wire Wire Line
+	2430 5060 2520 5060
+Wire Wire Line
+	2630 5000 2630 5060
+Connection ~ 2520 5060
+Wire Wire Line
+	2520 5060 2630 5060
+Wire Wire Line
+	3930 4840 3930 4760
+Wire Wire Line
+	3680 4850 3680 4760
+Wire Wire Line
+	3930 4760 3790 4760
+Wire Wire Line
+	3680 5050 3680 5170
+Wire Wire Line
+	3680 5170 3820 5170
+Wire Wire Line
+	3930 5170 3930 5040
+$Comp
+L power:+3V3 #PWR07
+U 1 1 5C1FC567
+P 3790 4760
+F 0 "#PWR07" H 3790 4610 50  0001 C CNN
+F 1 "+3V3" H 3805 4933 50  0000 C CNN
+F 2 "" H 3790 4760 50  0001 C CNN
+F 3 "" H 3790 4760 50  0001 C CNN
+	1    3790 4760
+	1    0    0    -1
+$EndComp
+Connection ~ 3790 4760
+Wire Wire Line
+	3790 4760 3680 4760
+$Comp
+L power:GND #PWR08
+U 1 1 5C1FC598
+P 3820 5170
+F 0 "#PWR08" H 3820 4920 50  0001 C CNN
+F 1 "GND" H 3825 4997 50  0000 C CNN
+F 2 "" H 3820 5170 50  0001 C CNN
+F 3 "" H 3820 5170 50  0001 C CNN
+	1    3820 5170
+	1    0    0    -1
+$EndComp
+Connection ~ 3820 5170
+Wire Wire Line
+	3820 5170 3930 5170
+$Comp
+L Device:C_Small C20
+U 1 1 5C20DCCF
+P 4870 4950
+F 0 "C20" H 4778 4904 50  0000 R CNN
+F 1 "C_Small" H 4778 4995 50  0000 R CNN
+F 2 "Capacitor_THT:CP_Radial_D10.0mm_P2.50mm_P5.00mm" H 4870 4950 50  0001 C CNN
+F 3 "~" H 4870 4950 50  0001 C CNN
+	1    4870 4950
+	1    0    0    1
+$EndComp
+$Comp
+L power:VCC #PWR011
+U 1 1 5C20DD11
+P 4870 4850
+F 0 "#PWR011" H 4870 4700 50  0001 C CNN
+F 1 "VCC" H 4887 5023 50  0000 C CNN
+F 2 "" H 4870 4850 50  0001 C CNN
+F 3 "" H 4870 4850 50  0001 C CNN
+	1    4870 4850
+	1    0    0    -1
+$EndComp
+$Comp
+L power:GND #PWR012
+U 1 1 5C20DD2A
+P 4870 5050
+F 0 "#PWR012" H 4870 4800 50  0001 C CNN
+F 1 "GND" H 4875 4877 50  0000 C CNN
+F 2 "" H 4870 5050 50  0001 C CNN
+F 3 "" H 4870 5050 50  0001 C CNN
+	1    4870 5050
+	1    0    0    -1
+$EndComp
 $EndSCHEMATC

Commit message: pic
pic controller en co gerouted
Parts:
- added D1, D2: 1N4004, Diode_THT:D_DO-41_SOD81_P10.16mm_Horizontal, symbol Diode:1N4004
- added J2: Barrel_Jack, Connector_BarrelJack:BarrelJack_Horizontal, symbol Connector:Barrel_Jack
Connections:
- wire segments 21 -> 33
Changed lines of the file:
@@
 L Connector:Screw_Terminal_01x02 J1
 U 1 1 5C194791
-P 2310 3100
-F 0 "J1" V 2290 2890 50  0000 C CNN
-F 1 "Screw_Terminal_01x02" V 2390 3070 50  0000 C CNN
-F 2 "TerminalBlock_Phoenix:TerminalBlock_Phoenix_MKDS-1,5-2-5.08_1x02_P5.08mm_Horizontal" H 2310 3100 50  0001 C CNN
-F 3 "~" H 2310 3100 50  0001 C CNN
-	1    2310 3100
+P 1850 3110
+F 0 "J1" V 1830 2900 50  0000 C CNN
+F 1 "Screw_Terminal_01x02" V 1930 3080 50  0000 C CNN
+F 2 "TerminalBlock_Phoenix:TerminalBlock_Phoenix_MKDS-1,5-2-5.08_1x02_P5.08mm_Horizontal" H 1850 3110 50  0001 C CNN
+F 3 "~" H 1850 3110 50  0001 C CNN
+	1    1850 3110
 	-1   0    0    1
 $EndComp
@@
 Wire Wire Line
 	2880 3000 3440 3000
-Wire Wire Line
-	2510 3100 2880 3100
 Wire Wire Line
 	2880 3100 2880 3340
@@
 	1    0    0    -1
 $EndComp
+$Comp
+L Connector:Barrel_Jack J2
+U 1 1 5C28AB96
+P 1420 4050
+F 0 "J2" H 1498 4375 50  0000 C CNN
+F 1 "Barrel_Jack" H 1498 4284 50  0000 C CNN
+F 2 "Connector_BarrelJack:BarrelJack_Horizontal" H 1470 4010 50  0001 C CNN
+F 3 "~" H 1470 4010 50  0001 C CNN
+	1    1420 4050
+	1    0    0    -1
+$EndComp
+$Comp
+L power:GND #PWR0132
+U 1 1 5C28AC5F
+P 1980 4180
+F 0 "#PWR0132" H 1980 3930 50  0001 C CNN
+F 1 "GND" H 1985 4007 50  0000 C CNN
+F 2 "" H 1980 4180 50  0001 C CNN
+F 3 "" H 1980 4180 50  0001 C CNN
+	1    1980 4180
+	1    0    0    -1
+$EndComp
+Wire Wire Line
+	1720 3950 2010 3950
+Wire Wire Line
+	1720 4050 1980 4050
+Wire Wire Line
+	1980 4050 1980 4150
+Wire Wire Line
+	1720 4150 1980 4150
+Connection ~ 1980 4150
+Wire Wire Line
+	1980 4150 1980 4180
+$Comp
+L Diode:1N4004 D2
+U 1 1 5C28C362
+P 2360 3000
+F 0 "D2" H 2360 2784 50  0000 C CNN
+F 1 "1N4004" H 2360 2875 50  0000 C CNN
+F 2 "Diode_THT:D_DO-41_SOD81_P10.16mm_Horizontal" H 2360 2825 50  0001 C CNN
+F 3 "http://www.vishay.com/docs/88503/1n4001.pdf" H 2360 3000 50  0001 C CNN
+	1    2360 3000
+	-1   0    0    1
+$EndComp
+Wire Wire Line
+	2050 3010 2160 3010
+Wire Wire Line
+	2160 3010 2160 3000
+Wire Wire Line
+	2160 3000 2210 3000
+Wire Wire Line
+	2050 3110 2470 3110
+Wire Wire Line
+	2470 3110 2470 3100
+Wire Wire Line
+	2470 3100 2880 3100
+$Comp
+L power:VCC #PWR013
+U 1 1 5C28CD78
+P 2460 3870
+F 0 "#PWR013" H 2460 3720 50  0001 C CNN
+F 1 "VCC" H 2477 4043 50  0000 C CNN
+F 2 "" H 2460 3870 50  0001 C CNN
+F 3 "" H 2460 3870 50  0001 C CNN
+	1    2460 3870
+	1    0    0    -1
+$EndComp
+$Comp
+L Diode:1N4004 D1
+U 1 1 5C28CCCC
+P 2160 3950
+F 0 "D1" H 2160 3734 50  0000 C CNN
+F 1 "1N4004" H 2160 3825 50  0000 C CNN
+F 2 "Diode_THT:D_DO-41_SOD81_P10.16mm_Horizontal" H 2160 3775 50  0001 C CNN
+F 3 "http://www.vishay.com/docs/88503/1n4001.pdf" H 2160 3950 50  0001 C CNN
+	1    2160 3950
+	-1   0    0    1
+$EndComp
+Wire Wire Line
+	2310 3950 2460 3950
+Wire Wire Line
+	2460 3950 2460 3870
 $EndSCHEMATC
